File: USB_HUB_4Port/USB_HUB_4Port.kicad_sch (KiCad schematic)
At the start: 33 parts, among them J1 HOST USB, J2 USB_A_4, J3 USB_A_3, J4 USB_A_2, J5 USB_A_1, J6 Jack-DC, U1 GL852G, Y1 12Mhz

Commit message: Add project 4 hub usb
Parts:
- U1: footprint Package_DFN_QFN:QFN-28-1EP_4x4mm_P0.45mm_EP2.4x2.4mm -> Package_DFN_QFN:QFN-28-1EP_5x5mm_P0.5mm_EP3.1x3.1mm
Changed lines of the file:
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@@
 			)
 		)
-		(property "Footprint" "Package_DFN_QFN:QFN-28-1EP_4x4mm_P0.45mm_EP2.4x2.4mm"
+		(property "Footprint" "Package_DFN_QFN:QFN-28-1EP_5x5mm_P0.5mm_EP3.1x3.1mm"
 			(at 132.08 57.15 0)
 			(effects
